File: PCBs/BMSBoard.brd (EAGLE design)
At the start: 100 x 80 mm, 33 parts, among them IC1 78L05Z, J1 12V, J2 24v_12v_gnd, J3 12V, J4 Switch-12V, J5 Switch-24V

Commit message: updated
Parts:
- removed U$1: DC-DC-STEP-DOWN-LM2596, diy-modules:DC-DC-STEP-DOWN-LM2596
- added IC2: LM2596S, national-semiconductor:TO263-5
Connections:
- removed net N$7: DFMINI.1, DUALMAX485.1, EXTRA1.1, EXTRA2.1, NANDGATE.1, NODEMCU.1, U$1.OUT+
- new net 24V: F3.1, IC2.1, J2.2, R3.1
- new net N$17: IC2.2
- new net N$18: IC2.4
- net GND: now also IC2.3; no longer U$1.IN-, U$1.OUT-
- net N$13: now also IC2.5; no longer F3.1, J2.2, R3.1, U$1.IN+
Changed lines of the file:
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@@
 <class number="0" name="default" width="0" drill="0">
+</class>
+<class number="1" name="New Class" width="0" drill="0">
 </class>
 </classes>
@@
 <attribute name="VALUE" x="-46.99" y="81.28" size="0.6096" layer="27" font="vector" ratio="20"/>
 </element>
-<element name="U$1" library="diy-modules" package="DC-DC-STEP-DOWN-LM2596" value="DC-DC-STEP-DOWN-LM2596" x="-35.56" y="13.97" smashed="yes">
-<attribute name="NAME" x="-35.56" y="25.4" size="1.27" layer="25" align="bottom-center"/>
-<attribute name="VALUE" x="-35.56" y="2.54" size="1.27" layer="27" align="top-center"/>
-</element>
 <element name="VOLTAGE-READ" library="Rembrandt Electronics - JST XH Connectors v1-0" package="JST-XH-02-PACKAGE-LONG-PAD" value="JST-XH-02-PIN-LONG-PAD" x="-77.47" y="30.48" smashed="yes">
 <attribute name="NAME" x="-81.725" y="28.44" size="1.016" layer="25" ratio="10" rot="R90"/>
 <attribute name="VALUE" x="-80.7725" y="34.3725" size="1.016" layer="27" ratio="10"/>
+</element>
+<element name="IC2" library="national-semiconductor" library_urn="urn:adsk.eagle:library:307" package="TO263-5" package3d_urn="urn:adsk.eagle:package:16438/2" value="LM2596S" x="-91.44" y="7.62" smashed="yes">
+<attribute name="MF" value="NATIONAL SEMICONDUCTOR" x="-91.44" y="7.62" size="1.778" layer="27" display="off"/>
+<attribute name="MPN" value="LM2596S-ADJ/NOPB" x="-91.44" y="7.62" size="1.778" layer="27" display="off"/>
+<attribute name="NAME" x="-97.028" y="2.032" size="1.27" layer="25" rot="R90"/>
+<attribute name="OC_FARNELL" value="9494367" x="-91.44" y="7.62" size="1.778" layer="27" display="off"/>
+<attribute name="OC_NEWARK" value="41K3842" x="-91.44" y="7.62" size="1.778" layer="27" display="off"/>
+<attribute name="POPULARITY" value="12" x="-91.44" y="7.62" size="1.778" layer="27" display="off"/>
+<attribute name="VALUE" x="-84.582" y="2.032" size="1.27" layer="27" rot="R90"/>
 </element>
 </elements>
@@
 <contactref element="RIGHTMOTOR24V" pad="1"/>
 <contactref element="LEFTMOTOR24V" pad="1"/>
-<contactref element="U$1" pad="IN-"/>
 <contactref element="NODEMCU" pad="2"/>
 <contactref element="DFMINI" pad="2"/>
@@
 <contactref element="EXTRA1" pad="2"/>
 <contactref element="EXTRA2" pad="2"/>
-<contactref element="U$1" pad="OUT-"/>
+<contactref element="IC2" pad="3"/>
+<wire x1="-72.41" y1="17.43" x2="-91.44" y2="1.8288" width="0" layer="19" extent="1-1"/>
 <wire x1="-78.74" y1="30.48" x2="-72.41" y2="17.43" width="0" layer="19" extent="1-1"/>
 <wire x1="-59.69" y1="29.71" x2="-72.41" y2="17.43" width="0" layer="19" extent="1-1"/>
@@
 <wire x1="-26.67" y1="60.96" x2="-26.67" y2="69.85" width="0" layer="19" extent="1-1"/>
 <wire x1="-27.96" y1="32.1" x2="-46.99" y2="30.48" width="0" layer="19" extent="1-1"/>
-<wire x1="-55.372" y1="5.334" x2="-72.41" y2="17.43" width="0" layer="19" extent="1-1"/>
-<wire x1="-15.748" y1="5.334" x2="-27.96" y2="32.1" width="0" layer="19" extent="1-1"/>
 </signal>
 <signal name="N$5">
@@
 <wire x1="-55.88" y1="28.71" x2="-13.97" y2="85.09" width="0" layer="19" extent="1-1"/>
 </signal>
-<signal name="N$13">
+<signal name="24V" class="1">
 <contactref element="F3" pad="1"/>
 <contactref element="J2" pad="2"/>
 <contactref element="R3" pad="1"/>
-<contactref element="U$1" pad="IN+"/>
-<wire x1="-43.26" y1="71.12" x2="-16.51" y2="85.09" width="0" layer="19" extent="1-1"/>
-<wire x1="-30.48" y1="50.8" x2="-43.26" y2="71.12" width="0" layer="19" extent="1-1"/>
-<wire x1="-55.372" y1="22.606" x2="-30.48" y2="50.8" width="0" layer="19" extent="1-1"/>
-</signal>
-<signal name="N$7">
-<contactref element="U$1" pad="OUT+"/>
-<contactref element="NODEMCU" pad="1"/>
-<contactref element="DFMINI" pad="1"/>
-<contactref element="DUALMAX485" pad="1"/>
-<contactref element="NANDGATE" pad="1"/>
-<contactref element="EXTRA1" pad="1"/>
-<contactref element="EXTRA2" pad="1"/>
-<wire x1="-29.21" y1="60.96" x2="-29.21" y2="69.85" width="0" layer="19" extent="1-1"/>
-<wire x1="-50.8" y1="60.96" x2="-29.21" y2="60.96" width="0" layer="19" extent="1-1"/>
-<wire x1="-49.53" y1="48.26" x2="-50.8" y2="60.96" width="0" layer="19" extent="1-1"/>
-<wire x1="-71.12" y1="48.26" x2="-49.53" y2="48.26" width="0" layer="19" extent="1-1"/>
-<wire x1="-72.39" y1="60.96" x2="-71.12" y2="48.26" width="0" layer="19" extent="1-1"/>
-<wire x1="-15.748" y1="22.606" x2="-29.21" y2="60.96" width="0" layer="19" extent="1-1"/>
+<contactref element="IC2" pad="1"/>
+<wire x1="-30.48" y1="50.8" x2="-94.8436" y2="1.8288" width="0" layer="19" extent="1-1"/>
+<wire x1="-43.26" y1="71.12" x2="-30.48" y2="50.8" width="0" layer="19" extent="1-1"/>
+<wire x1="-16.51" y1="85.09" x2="-43.26" y2="71.12" width="0" layer="19" extent="1-1"/>
+</signal>
+<signal name="N$13">
+<contactref element="IC2" pad="5"/>
+</signal>
+<signal name="N$17">
+<contactref element="IC2" pad="2"/>
+</signal>
+<signal name="N$18">
+<contactref element="IC2" pad="4"/>
 </signal>
 </signals>
