File: PCBs/BMSBoard.sch (EAGLE design)
At the start: 33 parts, among them IC1 78L05Z, J1 12V, J2 24v_12v_gnd, J3 12V, J4 Switch-12V, J5 Switch-24V

Commit message: updated
Parts:
- removed U$1: DC-DC-STEP-DOWN-LM2596, diy-modules:DC-DC-STEP-DOWN-LM2596
- added IC2: LM2596S, national-semiconductor:LM2596S
Connections:
- removed net N$7: DFMINI-1.S, DUALMAX485-1.S, EXTRA1-1.S, EXTRA2-1.S, NANDGATE-1.S, NODEMCU-1.S, U$1.OUT+
- new net 24V: F3.1, IC2.VIN, J2.2, R3.1
- new net N$17: IC2.OUT
- new net N$18: IC2.FB
- net GND: now also IC2.GND; no longer U$1.IN-, U$1.OUT-
- net N$13: now also IC2.!ON!/OFF; no longer F3.1, J2.2, R3.1, U$1.IN+
Changed lines of the file:
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@@
 <class number="0" name="default" width="0" drill="0">
+</class>
+<class number="1" name="New Class" width="0" drill="0">
 </class>
 </classes>
@@
 <part name="SUPPLY2" library="supply2" library_urn="urn:adsk.eagle:library:372" deviceset="GND" device=""/>
 <part name="SUPPLY15" library="supply2" library_urn="urn:adsk.eagle:library:372" deviceset="GND" device=""/>
-<part name="U$1" library="diy-modules" deviceset="DC-DC-STEP-DOWN-LM2596" device=""/>
-<part name="SUPPLY16" library="supply2" library_urn="urn:adsk.eagle:library:372" deviceset="GND" device=""/>
 <part name="NODEMCU" library="Rembrandt Electronics - JST XH Connectors v1-0" deviceset="JST-XH-02-PIN" device="-LONG-PAD"/>
 <part name="DFMINI" library="Rembrandt Electronics - JST XH Connectors v1-0" deviceset="JST-XH-02-PIN" device="-LONG-PAD"/>
@@
 <part name="SUPPLY21" library="supply2" library_urn="urn:adsk.eagle:library:372" deviceset="GND" device=""/>
 <part name="SUPPLY22" library="supply2" library_urn="urn:adsk.eagle:library:372" deviceset="GND" device=""/>
-<part name="SUPPLY23" library="supply2" library_urn="urn:adsk.eagle:library:372" deviceset="GND" device=""/>
+<part name="SUPPLY25" library="supply2" library_urn="urn:adsk.eagle:library:372" deviceset="GND" device=""/>
+<part name="IC2" library="national-semiconductor" library_urn="urn:adsk.eagle:library:307" deviceset="LM2596" device="S" package3d_urn="urn:adsk.eagle:package:16438/2"/>
 </parts>
 <sheets>
@@
 <attribute name="VALUE" x="46.355" y="3.175" size="1.778" layer="96" rot="R90"/>
 </instance>
-<instance part="U$1" gate="G$1" x="152.4" y="2.54" smashed="yes">
-<attribute name="NAME" x="139.7" y="17.78" size="1.778" layer="95"/>
-<attribute name="VALUE" x="139.7" y="15.24" size="1.778" layer="96"/>
-</instance>
-<instance part="SUPPLY16" gate="GND" x="134.62" y="-5.08" smashed="yes">
-<attribute name="VALUE" x="132.715" y="-8.255" size="1.778" layer="96"/>
-</instance>
 <instance part="NODEMCU" gate="-2" x="185.42" y="22.86" smashed="yes">
 <attribute name="NAME" x="187.96" y="22.098" size="1.524" layer="95"/>
@@
 <attribute name="VALUE" x="180.975" y="-23.495" size="1.778" layer="96"/>
 </instance>
-<instance part="SUPPLY23" gate="GND" x="170.18" y="-5.08" smashed="yes">
-<attribute name="VALUE" x="168.275" y="-8.255" size="1.778" layer="96"/>
+<instance part="SUPPLY25" gate="GND" x="134.62" y="-55.88" smashed="yes">
+<attribute name="VALUE" x="132.715" y="-59.055" size="1.778" layer="96"/>
+</instance>
+<instance part="IC2" gate="G$1" x="93.98" y="-10.16" smashed="yes">
+<attribute name="NAME" x="83.82" y="-1.27" size="1.778" layer="95"/>
+<attribute name="VALUE" x="83.82" y="-20.32" size="1.778" layer="96"/>
 </instance>
 </instances>
@@
 </segment>
 <segment>
-<pinref part="U$1" gate="G$1" pin="IN-"/>
-<pinref part="SUPPLY16" gate="GND" pin="GND"/>
-</segment>
-<segment>
 <pinref part="NODEMCU" gate="-2" pin="S"/>
 <pinref part="SUPPLY17" gate="GND" pin="GND"/>
@@
 </segment>
 <segment>
-<pinref part="U$1" gate="G$1" pin="OUT-"/>
-<pinref part="SUPPLY23" gate="GND" pin="GND"/>
+<pinref part="IC2" gate="G$1" pin="GND"/>
+<wire x1="81.28" y1="-15.24" x2="73.66" y2="-15.24" width="0.1524" layer="91"/>
+<label x="73.66" y="-15.24" size="1.778" layer="95"/>
 </segment>
 </net>
@@
 </segment>
 </net>
-<net name="N$13" class="0">
-<segment>
+<net name="24V" class="1">
+<segment>
+<pinref part="R3" gate="G$1" pin="1"/>
+<wire x1="88.9" y1="25.4" x2="109.22" y2="25.4" width="0.1524" layer="91"/>
+<wire x1="88.9" y1="22.86" x2="88.9" y2="25.4" width="0.1524" layer="91"/>
 <pinref part="F3" gate="F" pin="1"/>
+<wire x1="76.2" y1="22.86" x2="88.9" y2="22.86" width="0.1524" layer="91"/>
+<junction x="76.2" y="22.86"/>
 <pinref part="J2" gate="J$1" pin="2"/>
 <wire x1="76.2" y1="20.32" x2="76.2" y2="22.86" width="0.1524" layer="91"/>
-<wire x1="76.2" y1="22.86" x2="88.9" y2="22.86" width="0.1524" layer="91"/>
-<wire x1="88.9" y1="22.86" x2="88.9" y2="25.4" width="0.1524" layer="91"/>
-<junction x="76.2" y="22.86"/>
-<pinref part="R3" gate="G$1" pin="1"/>
-<wire x1="88.9" y1="25.4" x2="93.98" y2="25.4" width="0.1524" layer="91"/>
-<wire x1="93.98" y1="25.4" x2="109.22" y2="25.4" width="0.1524" layer="91"/>
-<wire x1="93.98" y1="25.4" x2="93.98" y2="2.54" width="0.1524" layer="91"/>
-<junction x="93.98" y="25.4"/>
-<pinref part="U$1" gate="G$1" pin="IN+"/>
-<wire x1="93.98" y1="2.54" x2="134.62" y2="2.54" width="0.1524" layer="91"/>
-<wire x1="134.62" y1="2.54" x2="134.62" y2="7.62" width="0.1524" layer="91"/>
-</segment>
-</net>
-<net name="N$7" class="0">
-<segment>
-<pinref part="U$1" gate="G$1" pin="OUT+"/>
-<wire x1="170.18" y1="7.62" x2="170.18" y2="10.16" width="0.1524" layer="91"/>
-<wire x1="170.18" y1="10.16" x2="170.18" y2="17.78" width="0.1524" layer="91"/>
-<wire x1="170.18" y1="17.78" x2="170.18" y2="25.4" width="0.1524" layer="91"/>
-<wire x1="170.18" y1="25.4" x2="182.88" y2="25.4" width="0.1524" layer="91"/>
-<pinref part="NODEMCU" gate="-1" pin="S"/>
-<pinref part="DFMINI" gate="-1" pin="S"/>
-<wire x1="182.88" y1="17.78" x2="170.18" y2="17.78" width="0.1524" layer="91"/>
-<junction x="170.18" y="17.78"/>
-<pinref part="DUALMAX485" gate="-1" pin="S"/>
-<wire x1="182.88" y1="10.16" x2="172.72" y2="10.16" width="0.1524" layer="91"/>
-<junction x="170.18" y="10.16"/>
-<pinref part="NANDGATE" gate="-1" pin="S"/>
-<wire x1="172.72" y1="10.16" x2="170.18" y2="10.16" width="0.1524" layer="91"/>
-<wire x1="182.88" y1="2.54" x2="177.8" y2="2.54" width="0.1524" layer="91"/>
-<wire x1="175.26" y1="2.54" x2="172.72" y2="2.54" width="0.1524" layer="91"/>
-<wire x1="172.72" y1="2.54" x2="172.72" y2="10.16" width="0.1524" layer="91"/>
-<junction x="172.72" y="10.16"/>
-<pinref part="EXTRA1" gate="-1" pin="S"/>
-<wire x1="182.88" y1="-5.08" x2="177.8" y2="-5.08" width="0.1524" layer="91"/>
-<wire x1="177.8" y1="-5.08" x2="177.8" y2="2.54" width="0.1524" layer="91"/>
-<wire x1="177.8" y1="2.54" x2="175.26" y2="2.54" width="0.1524" layer="91"/>
-<pinref part="EXTRA2" gate="-1" pin="S"/>
-<wire x1="182.88" y1="-15.24" x2="175.26" y2="-15.24" width="0.1524" layer="91"/>
-<wire x1="175.26" y1="-15.24" x2="175.26" y2="2.54" width="0.1524" layer="91"/>
-<junction x="175.26" y="2.54"/>
-</segment>
-</net>
+<label x="96.52" y="20.32" size="1.778" layer="95"/>
+</segment>
+<segment>
+<pinref part="IC2" gate="G$1" pin="VIN"/>
+<wire x1="81.28" y1="-5.08" x2="73.66" y2="-5.08" width="0.1524" layer="91"/>
+<label x="73.66" y="-5.08" size="1.778" layer="95"/>
+</segment>
+</net>
+<net name="N$13" class="0">
+<segment>
+<pinref part="IC2" gate="G$1" pin="!ON!/OFF"/>
+<wire x1="81.28" y1="-10.16" x2="73.66" y2="-10.16" width="0.1524" layer="91"/>
+</segment>
+</net>
+<net name="N$17" class="0">
+<segment>
+<pinref part="IC2" gate="G$1" pin="OUT"/>
+<wire x1="106.68" y1="-7.62" x2="111.76" y2="-7.62" width="0.1524" layer="91"/>
+</segment>
+</net>
+<net name="N$18" class="0">
+<segment>
+<pinref part="IC2" gate="G$1" pin="FB"/>
+<wire x1="106.68" y1="-12.7" x2="111.76" y2="-12.7" width="0.1524" layer="91"/>
+</segment>
+</net>
