File: PCBs/DualMax485.sch (EAGLE design)
At the start: 14 parts, among them IC2 7805DT, J1 6V-12V

Commit message: updated something
Connections:
- new net N$16: IC2.VI, J1.1
- net VCC: no longer IC2.VI, J1.1
Changed lines of the file:
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@@
 <part name="SUPPLY6" library="supply2" library_urn="urn:adsk.eagle:library:372" deviceset="GND" device=""/>
 <part name="SUPPLY12" library="supply2" library_urn="urn:adsk.eagle:library:372" deviceset="GND" device=""/>
-<part name="SUPPLY14" library="supply2" library_urn="urn:adsk.eagle:library:372" deviceset="VCC" device=""/>
 <part name="SUPPLY2" library="supply2" library_urn="urn:adsk.eagle:library:372" deviceset="VCC" device=""/>
 <part name="SUPPLY3" library="supply2" library_urn="urn:adsk.eagle:library:372" deviceset="GND" device=""/>
 <part name="SUPPLY1" library="supply2" library_urn="urn:adsk.eagle:library:372" deviceset="VCC" device=""/>
 <part name="J1" library="SparkFun-Connectors" deviceset="CONN_02" device="5MM" value="6V-12V"/>
-<part name="SUPPLY10" library="supply2" library_urn="urn:adsk.eagle:library:372" deviceset="VCC" device=""/>
 <part name="SUPPLY13" library="supply2" library_urn="urn:adsk.eagle:library:372" deviceset="GND" device=""/>
 <part name="LED1" library="adafruit" deviceset="LED" device="CHIPLED_0805" value="Red"/>
@@
 <attribute name="VALUE" x="-81.915" y="130.175" size="1.778" layer="96" rot="R180"/>
 </instance>
-<instance part="SUPPLY14" gate="G$1" x="-71.12" y="116.84" smashed="yes" rot="R270">
-<attribute name="VALUE" x="-65.405" y="123.825" size="1.778" layer="96" rot="R270"/>
-</instance>
 <instance part="SUPPLY2" gate="G$1" x="-22.86" y="106.68" smashed="yes">
 <attribute name="VALUE" x="-24.765" y="89.535" size="1.778" layer="96"/>
 </instance>
-<instance part="SUPPLY3" gate="GND" x="-15.24" y="93.98" smashed="yes">
-<attribute name="VALUE" x="-17.145" y="90.805" size="1.778" layer="96"/>
-</instance>
-<instance part="SUPPLY1" gate="G$1" x="-96.52" y="116.84" smashed="yes" rot="R90">
-<attribute name="VALUE" x="-99.695" y="114.935" size="1.778" layer="96" rot="R90"/>
+<instance part="SUPPLY3" gate="GND" x="-10.16" y="93.98" smashed="yes">
+<attribute name="VALUE" x="-12.065" y="90.805" size="1.778" layer="96"/>
+</instance>
+<instance part="SUPPLY1" gate="G$1" x="-106.68" y="116.84" smashed="yes" rot="R90">
+<attribute name="VALUE" x="-109.855" y="114.935" size="1.778" layer="96" rot="R90"/>
 </instance>
 <instance part="J1" gate="G$1" x="-96.52" y="104.14" smashed="yes" rot="R180">
@@
 <attribute name="NAME" x="-93.98" y="98.552" size="1.778" layer="95" font="vector" rot="R180"/>
 </instance>
-<instance part="SUPPLY10" gate="G$1" x="-104.14" y="106.68" smashed="yes"/>
 <instance part="SUPPLY13" gate="GND" x="-104.14" y="99.06" smashed="yes">
 <attribute name="VALUE" x="-106.045" y="95.885" size="1.778" layer="96"/>
@@
 <net name="VCC" class="0">
 <segment>
-<pinref part="J1" gate="G$1" pin="1"/>
-<pinref part="SUPPLY10" gate="G$1" pin="VCC"/>
-</segment>
-<segment>
 <pinref part="R1" gate="G$1" pin="1"/>
 <pinref part="SUPPLY15" gate="G$1" pin="VCC"/>
-</segment>
-<segment>
-<pinref part="SUPPLY14" gate="G$1" pin="VCC"/>
-<pinref part="IC2" gate="A1" pin="VI"/>
 </segment>
 <segment>
@@
 <pinref part="5V" gate="-1" pin="S"/>
 <wire x1="-104.14" y1="121.92" x2="-104.14" y2="116.84" width="0.1524" layer="91"/>
+<junction x="-104.14" y="116.84"/>
 <wire x1="-104.14" y1="116.84" x2="-93.98" y2="116.84" width="0.1524" layer="91"/>
-<junction x="-93.98" y="116.84"/>
 </segment>
 <segment>
@@
 <pinref part="SUPPLY3" gate="GND" pin="GND"/>
 <pinref part="RS485OUTCONNECTEDTOD-D+GND" gate="-3" pin="S"/>
-<wire x1="-15.24" y1="96.52" x2="12.7" y2="96.52" width="0.1524" layer="91"/>
-<wire x1="-15.24" y1="96.52" x2="-22.86" y2="96.52" width="0.1524" layer="91"/>
+<wire x1="-10.16" y1="96.52" x2="12.7" y2="96.52" width="0.1524" layer="91"/>
+<wire x1="-10.16" y1="96.52" x2="-22.86" y2="96.52" width="0.1524" layer="91"/>
+<junction x="-10.16" y="96.52"/>
 </segment>
 <segment>
@@
 </segment>
 </net>
+<net name="N$16" class="0">
+<segment>
+<pinref part="IC2" gate="A1" pin="VI"/>
+<wire x1="-73.66" y1="116.84" x2="-68.58" y2="116.84" width="0.1524" layer="91"/>
+<wire x1="-68.58" y1="116.84" x2="-68.58" y2="109.22" width="0.1524" layer="91"/>
+<wire x1="-68.58" y1="109.22" x2="-104.14" y2="109.22" width="0.1524" layer="91"/>
+<pinref part="J1" gate="G$1" pin="1"/>
+<wire x1="-104.14" y1="109.22" x2="-104.14" y2="104.14" width="0.1524" layer="91"/>
+</segment>
+</net>
 </nets>
 </sheet>
 </sheets>
-<errors>
-</errors>
 </schematic>
 </drawing>

Commit message: board updated
Parts:
- added C1: 0.1uF, adafruit:C-USC0805
- added C2: 0.22uF, adafruit:C-USC0805
- J1: value 6V-12V -> 7V-9V
- renumbered RS485CONNECTEDTOD-D+GND to DRIVERD-D+GND, RS485OUTCONNECTEDTOD-D+GND to D-D+GND
Connections:
- net GND: now also C1.2, C2.2
- net N$16: now also C2.1
- net VCC: now also C1.1
Changed lines of the file:
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@@
 <part name="SUPPLY3" library="supply2" library_urn="urn:adsk.eagle:library:372" deviceset="GND" device=""/>
 <part name="SUPPLY1" library="supply2" library_urn="urn:adsk.eagle:library:372" deviceset="VCC" device=""/>
-<part name="J1" library="SparkFun-Connectors" deviceset="CONN_02" device="5MM" value="6V-12V"/>
+<part name="J1" library="SparkFun-Connectors" deviceset="CONN_02" device="5MM" value="7V-9V"/>
 <part name="SUPPLY13" library="supply2" library_urn="urn:adsk.eagle:library:372" deviceset="GND" device=""/>
 <part name="LED1" library="adafruit" deviceset="LED" device="CHIPLED_0805" value="Red"/>
@@
 <part name="R4" library="adafruit" deviceset="R-US_" device="M0805" value="1k"/>
 <part name="R5" library="adafruit" deviceset="R-US_" device="M0805" value="1k"/>
-<part name="RS485OUTCONNECTEDTOD-D+GND" library="Rembrandt Electronics - JST XH Connectors v1-0" deviceset="JST-XH-03-PIN" device="-LONG-PAD"/>
-<part name="RS485CONNECTEDTOD-D+GND" library="Rembrandt Electronics - JST XH Connectors v1-0" deviceset="JST-XH-03-PIN" device="-LONG-PAD"/>
+<part name="D-D+GND" library="Rembrandt Electronics - JST XH Connectors v1-0" deviceset="JST-XH-03-PIN" device="-LONG-PAD"/>
+<part name="DRIVERD-D+GND" library="Rembrandt Electronics - JST XH Connectors v1-0" deviceset="JST-XH-03-PIN" device="-LONG-PAD"/>
+<part name="C1" library="adafruit" deviceset="C-US" device="C0805" value="0.1uF"/>
+<part name="C2" library="adafruit" deviceset="C-US" device="C0805" value="0.22uF"/>
+<part name="SUPPLY4" library="supply2" library_urn="urn:adsk.eagle:library:372" deviceset="GND" device=""/>
+<part name="SUPPLY7" library="supply2" library_urn="urn:adsk.eagle:library:372" deviceset="GND" device=""/>
 </parts>
 <sheets>
@@
 <attribute name="VALUE" x="-82.55" y="67.818" size="1.778" layer="96"/>
 </instance>
-<instance part="RS485OUTCONNECTEDTOD-D+GND" gate="-1" x="15.24" y="101.6" smashed="yes">
+<instance part="D-D+GND" gate="-1" x="15.24" y="101.6" smashed="yes">
 <attribute name="NAME" x="17.78" y="100.838" size="1.524" layer="95"/>
 <attribute name="VALUE" x="14.478" y="102.997" size="1.778" layer="96"/>
 </instance>
-<instance part="RS485OUTCONNECTEDTOD-D+GND" gate="-2" x="15.24" y="99.06" smashed="yes">
+<instance part="D-D+GND" gate="-2" x="15.24" y="99.06" smashed="yes">
 <attribute name="NAME" x="17.78" y="98.298" size="1.524" layer="95"/>
 </instance>
-<instance part="RS485OUTCONNECTEDTOD-D+GND" gate="-3" x="15.24" y="96.52" smashed="yes">
+<instance part="D-D+GND" gate="-3" x="15.24" y="96.52" smashed="yes">
 <attribute name="NAME" x="17.78" y="95.758" size="1.524" layer="95"/>
 </instance>
-<instance part="RS485CONNECTEDTOD-D+GND" gate="-1" x="15.24" y="83.82" smashed="yes">
+<instance part="DRIVERD-D+GND" gate="-1" x="15.24" y="83.82" smashed="yes">
 <attribute name="NAME" x="17.78" y="83.058" size="1.524" layer="95"/>
 <attribute name="VALUE" x="14.478" y="85.217" size="1.778" layer="96"/>
 </instance>
-<instance part="RS485CONNECTEDTOD-D+GND" gate="-2" x="15.24" y="81.28" smashed="yes">
+<instance part="DRIVERD-D+GND" gate="-2" x="15.24" y="81.28" smashed="yes">
 <attribute name="NAME" x="17.78" y="80.518" size="1.524" layer="95"/>
 </instance>
-<instance part="RS485CONNECTEDTOD-D+GND" gate="-3" x="15.24" y="78.74" smashed="yes">
+<instance part="DRIVERD-D+GND" gate="-3" x="15.24" y="78.74" smashed="yes">
 <attribute name="NAME" x="17.78" y="77.978" size="1.524" layer="95"/>
+</instance>
+<instance part="C1" gate="G$1" x="-119.38" y="109.22" smashed="yes">
+<attribute name="NAME" x="-118.364" y="109.855" size="1.778" layer="95"/>
+<attribute name="VALUE" x="-118.364" y="105.029" size="1.778" layer="96"/>
+</instance>
+<instance part="C2" gate="G$1" x="-111.76" y="109.22" smashed="yes">
+<attribute name="NAME" x="-110.744" y="109.855" size="1.778" layer="95"/>
+<attribute name="VALUE" x="-110.744" y="105.029" size="1.778" layer="96"/>
+</instance>
+<instance part="SUPPLY4" gate="GND" x="-119.38" y="99.06" smashed="yes">
+<attribute name="VALUE" x="-121.285" y="95.885" size="1.778" layer="96"/>
+</instance>
+<instance part="SUPPLY7" gate="GND" x="-111.76" y="99.06" smashed="yes">
+<attribute name="VALUE" x="-113.665" y="95.885" size="1.778" layer="96"/>
 </instance>
 </instances>
@@
 <wire x1="-104.14" y1="121.92" x2="-104.14" y2="116.84" width="0.1524" layer="91"/>
 <junction x="-104.14" y="116.84"/>
-<wire x1="-104.14" y1="116.84" x2="-93.98" y2="116.84" width="0.1524" layer="91"/>
+<wire x1="-104.14" y1="116.84" x2="-99.06" y2="116.84" width="0.1524" layer="91"/>
+<wire x1="-99.06" y1="116.84" x2="-93.98" y2="116.84" width="0.1524" layer="91"/>
+<wire x1="-99.06" y1="116.84" x2="-99.06" y2="114.3" width="0.1524" layer="91"/>
+<junction x="-99.06" y="116.84"/>
+<wire x1="-99.06" y1="114.3" x2="-119.38" y2="114.3" width="0.1524" layer="91"/>
+<pinref part="C1" gate="G$1" pin="1"/>
+<wire x1="-119.38" y1="114.3" x2="-119.38" y2="111.76" width="0.1524" layer="91"/>
 </segment>
 <segment>
@@
 <pinref part="RS485MODULE2" gate="G$1" pin="GND"/>
 <pinref part="SUPPLY3" gate="GND" pin="GND"/>
-<pinref part="RS485OUTCONNECTEDTOD-D+GND" gate="-3" pin="S"/>
+<pinref part="D-D+GND" gate="-3" pin="S"/>
 <wire x1="-10.16" y1="96.52" x2="12.7" y2="96.52" width="0.1524" layer="91"/>
 <wire x1="-10.16" y1="96.52" x2="-22.86" y2="96.52" width="0.1524" layer="91"/>
@@
 <wire x1="-17.78" y1="76.2" x2="-2.54" y2="76.2" width="0.1524" layer="91"/>
 <wire x1="-2.54" y1="76.2" x2="-2.54" y2="78.74" width="0.1524" layer="91"/>
-<pinref part="RS485CONNECTEDTOD-D+GND" gate="-3" pin="S"/>
+<pinref part="DRIVERD-D+GND" gate="-3" pin="S"/>
 <wire x1="-2.54" y1="78.74" x2="12.7" y2="78.74" width="0.1524" layer="91"/>
 <wire x1="-17.78" y1="76.2" x2="-22.86" y2="76.2" width="0.1524" layer="91"/>
 <junction x="-17.78" y="76.2"/>
+</segment>
+<segment>
+<pinref part="SUPPLY7" gate="GND" pin="GND"/>
+<pinref part="C2" gate="G$1" pin="2"/>
+<wire x1="-111.76" y1="101.6" x2="-111.76" y2="104.14" width="0.1524" layer="91"/>
+</segment>
+<segment>
+<pinref part="SUPPLY4" gate="GND" pin="GND"/>
+<pinref part="C1" gate="G$1" pin="2"/>
+<wire x1="-119.38" y1="101.6" x2="-119.38" y2="104.14" width="0.1524" layer="91"/>
 </segment>
 </net>
@@
 <pinref part="RS485MODULE2" gate="G$1" pin="B"/>
 <wire x1="-22.86" y1="101.6" x2="12.7" y2="101.6" width="0.1524" layer="91"/>
-<pinref part="RS485OUTCONNECTEDTOD-D+GND" gate="-1" pin="S"/>
+<pinref part="D-D+GND" gate="-1" pin="S"/>
 </segment>
 </net>
@@
 <segment>
 <pinref part="RS485MODULE2" gate="G$1" pin="A"/>
-<pinref part="RS485OUTCONNECTEDTOD-D+GND" gate="-2" pin="S"/>
+<pinref part="D-D+GND" gate="-2" pin="S"/>
 <wire x1="-22.86" y1="99.06" x2="12.7" y2="99.06" width="0.1524" layer="91"/>
 </segment>
@@
 <net name="N$12" class="0">
 <segment>
-<pinref part="RS485CONNECTEDTOD-D+GND" gate="-1" pin="S"/>
+<pinref part="DRIVERD-D+GND" gate="-1" pin="S"/>
 <wire x1="-7.62" y1="83.82" x2="12.7" y2="83.82" width="0.1524" layer="91"/>
 <wire x1="-7.62" y1="81.28" x2="-7.62" y2="83.82" width="0.1524" layer="91"/>
@@
 <wire x1="-22.86" y1="78.74" x2="-5.08" y2="78.74" width="0.1524" layer="91"/>
 <wire x1="-5.08" y1="78.74" x2="-5.08" y2="81.28" width="0.1524" layer="91"/>
-<pinref part="RS485CONNECTEDTOD-D+GND" gate="-2" pin="S"/>
+<pinref part="DRIVERD-D+GND" gate="-2" pin="S"/>
 <wire x1="-5.08" y1="81.28" x2="12.7" y2="81.28" width="0.1524" layer="91"/>
 </segment>
@@
 <segment>
 <pinref part="IC2" gate="A1" pin="VI"/>
-<wire x1="-73.66" y1="116.84" x2="-68.58" y2="116.84" width="0.1524" layer="91"/>
+<wire x1="-73.66" y1="116.84" x2="-71.12" y2="116.84" width="0.1524" layer="91"/>
+<wire x1="-71.12" y1="116.84" x2="-68.58" y2="116.84" width="0.1524" layer="91"/>
 <wire x1="-68.58" y1="116.84" x2="-68.58" y2="109.22" width="0.1524" layer="91"/>
 <wire x1="-68.58" y1="109.22" x2="-104.14" y2="109.22" width="0.1524" layer="91"/>
 <pinref part="J1" gate="G$1" pin="1"/>
 <wire x1="-104.14" y1="109.22" x2="-104.14" y2="104.14" width="0.1524" layer="91"/>
-</segment>
-</net>
+<pinref part="C2" gate="G$1" pin="1"/>
+<wire x1="-111.76" y1="111.76" x2="-71.12" y2="111.76" width="0.1524" layer="91"/>
+<wire x1="-71.12" y1="111.76" x2="-71.12" y2="116.84" width="0.1524" layer="91"/>
+<junction x="-71.12" y="116.84"/>
+</segment>
+</net>
