File: PCBs/DualMax485.brd (EAGLE design)
At the start: 59.4 x 47 mm, 10 parts, among them IC2 7805DT, J1 6V-12V

Commit message: resistors added to max485
Parts:
- added R2, R3, R4, R5: 1k, adafruit:M0805
Connections:
- new net N$11: R2.1, RS232IN.7
- new net N$14: R4.2, RS485MODULE1.J1.4
- new net N$15: R5.2, RS485MODULE1.J1.1
- new net N$5: R3.1, RS232IN.5
- net N$10: now also R4.1; no longer RS485MODULE1.J1.4
- net N$2: now also R3.2; no longer RS232IN.5
- net N$3: now also R2.2; no longer RS232IN.7
- net N$8: now also R5.1; no longer RS485MODULE1.J1.1
Routing:
- net N$3: track 9.72 -> 2.54 mm
- net N$8: track 8.78 -> 3.49 mm
Changed lines of the file:
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@@
 <drawing>
 <settings>
-<setting alwaysvectorfont="yes"/>
+<setting alwaysvectorfont="no"/>
 <setting verticaltext="up"/>
 </settings>
@@
 <attribute name="VALUE" x="27.1775" y="69.9325" size="1.016" layer="27" ratio="10"/>
 </element>
+<element name="R2" library="adafruit" package="M0805" value="1k" x="2.54" y="21.59" smashed="yes">
+<attribute name="NAME" x="1.524" y="22.606" size="1.27" layer="25"/>
+<attribute name="VALUE" x="1.524" y="19.304" size="1.27" layer="27"/>
+</element>
+<element name="R3" library="adafruit" package="M0805" value="1k" x="2.54" y="15.24" smashed="yes">
+<attribute name="NAME" x="1.524" y="16.256" size="1.27" layer="25"/>
+<attribute name="VALUE" x="1.524" y="12.954" size="1.27" layer="27"/>
+</element>
+<element name="R4" library="adafruit" package="M0805" value="1k" x="2.54" y="8.89" smashed="yes">
+<attribute name="NAME" x="1.524" y="9.906" size="1.27" layer="25"/>
+<attribute name="VALUE" x="1.524" y="6.604" size="1.27" layer="27"/>
+</element>
+<element name="R5" library="adafruit" package="M0805" value="1k" x="2.54" y="2.54" smashed="yes">
+<attribute name="NAME" x="1.524" y="3.556" size="1.27" layer="25"/>
+<attribute name="VALUE" x="1.524" y="0.254" size="1.27" layer="27"/>
+</element>
 </elements>
 <signals>
@@
 </signal>
 <signal name="N$2">
-<contactref element="RS232IN" pad="5"/>
 <contactref element="RS485MODULE2" pad="J1.1"/>
 <wire x1="9.144" y1="49.3776" x2="13.716" y2="49.3776" width="0.6096" layer="1"/>
 <wire x1="6.4008" y1="46.6344" x2="9.144" y2="49.3776" width="0.6096" layer="1"/>
 <wire x1="13.716" y1="49.3776" x2="13.97" y2="49.53" width="0.6096" layer="1"/>
-<wire x1="6.4008" y1="46.6344" x2="6.35" y2="46.99" width="0.6096" layer="1"/>
+<contactref element="R3" pad="2"/>
+<wire x1="3.49" y1="15.24" x2="6.4008" y2="46.6344" width="0" layer="19" extent="1-1"/>
 </signal>
 <signal name="N$3">
-<contactref element="RS232IN" pad="7"/>
 <contactref element="RS485MODULE2" pad="J1.4"/>
 <wire x1="11.43" y1="57.15" x2="13.97" y2="57.15" width="0.6096" layer="1"/>
-<wire x1="6.35" y1="52.07" x2="11.43" y2="57.15" width="0.6096" layer="1"/>
+<contactref element="R2" pad="2"/>
+<wire x1="3.49" y1="21.59" x2="11.43" y2="57.15" width="0" layer="19" extent="1-1"/>
 </signal>
 <signal name="N$4">
@@
 <signal name="N$8">
 <contactref element="RS232IN" pad="1"/>
-<contactref element="RS485MODULE1" pad="J1.1"/>
-<wire x1="8.6868" y1="34.29" x2="13.97" y2="34.29" width="0.6096" layer="1"/>
 <wire x1="6.4008" y1="36.576" x2="8.6868" y2="34.29" width="0.6096" layer="1"/>
 <wire x1="6.4008" y1="36.576" x2="6.35" y2="36.83" width="0.6096" layer="1"/>
+<contactref element="R5" pad="1"/>
+<wire x1="1.59" y1="2.54" x2="8.6868" y2="34.29" width="0" layer="19" extent="1-1"/>
 </signal>
 <signal name="N$10">
 <contactref element="RS232IN" pad="3"/>
-<contactref element="RS485MODULE1" pad="J1.4"/>
 <wire x1="6.4008" y1="42.0624" x2="13.716" y2="42.0624" width="0.6096" layer="1"/>
-<wire x1="13.716" y1="42.0624" x2="13.97" y2="41.91" width="0.6096" layer="1"/>
 <wire x1="6.4008" y1="42.0624" x2="6.35" y2="41.91" width="0.6096" layer="1"/>
+<contactref element="R4" pad="1"/>
+<wire x1="1.59" y1="8.89" x2="6.35" y2="41.91" width="0" layer="19" extent="1-1"/>
 </signal>
 <signal name="N$12">
@@
 <wire x1="52.1208" y1="64.4652" x2="52.07" y2="64.77" width="0.6096" layer="1"/>
 </signal>
+<signal name="N$5">
+<contactref element="RS232IN" pad="5"/>
+<contactref element="R3" pad="1"/>
+<wire x1="1.59" y1="15.24" x2="6.35" y2="46.99" width="0" layer="19" extent="1-1"/>
+</signal>
+<signal name="N$11">
+<contactref element="RS232IN" pad="7"/>
+<contactref element="R2" pad="1"/>
+<wire x1="1.59" y1="21.59" x2="6.35" y2="52.07" width="0" layer="19" extent="1-1"/>
+</signal>
+<signal name="N$15">
+<contactref element="RS485MODULE1" pad="J1.1"/>
+<contactref element="R5" pad="2"/>
+<wire x1="3.49" y1="2.54" x2="13.97" y2="34.29" width="0" layer="19" extent="1-1"/>
+</signal>
+<signal name="N$14">
+<contactref element="RS485MODULE1" pad="J1.4"/>
+<contactref element="R4" pad="2"/>
+<wire x1="3.49" y1="8.89" x2="13.97" y2="41.91" width="0" layer="19" extent="1-1"/>
+</signal>
 </signals>

Commit message: updated
Parts:
- moved R5 29.6 mm to (17.8, 27.9)
- moved R4 21.6 mm to (12.7, 27.9)
- moved R3 13.7 mm to (7.62, 27.9)
- moved R2 10.2 mm to (7.62, 30.5)
Changed lines of the file:
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@@
 <attribute name="VALUE" x="27.1775" y="69.9325" size="1.016" layer="27" ratio="10"/>
 </element>
-<element name="R2" library="adafruit" package="M0805" value="1k" x="2.54" y="21.59" smashed="yes">
-<attribute name="NAME" x="1.524" y="22.606" size="1.27" layer="25"/>
-<attribute name="VALUE" x="1.524" y="19.304" size="1.27" layer="27"/>
-</element>
-<element name="R3" library="adafruit" package="M0805" value="1k" x="2.54" y="15.24" smashed="yes">
-<attribute name="NAME" x="1.524" y="16.256" size="1.27" layer="25"/>
-<attribute name="VALUE" x="1.524" y="12.954" size="1.27" layer="27"/>
-</element>
-<element name="R4" library="adafruit" package="M0805" value="1k" x="2.54" y="8.89" smashed="yes">
-<attribute name="NAME" x="1.524" y="9.906" size="1.27" layer="25"/>
-<attribute name="VALUE" x="1.524" y="6.604" size="1.27" layer="27"/>
-</element>
-<element name="R5" library="adafruit" package="M0805" value="1k" x="2.54" y="2.54" smashed="yes">
-<attribute name="NAME" x="1.524" y="3.556" size="1.27" layer="25"/>
-<attribute name="VALUE" x="1.524" y="0.254" size="1.27" layer="27"/>
+<element name="R2" library="adafruit" package="M0805" value="1k" x="7.62" y="30.48" smashed="yes">
+<attribute name="NAME" x="6.604" y="31.496" size="1.27" layer="25"/>
+<attribute name="VALUE" x="6.604" y="28.194" size="1.27" layer="27"/>
+</element>
+<element name="R3" library="adafruit" package="M0805" value="1k" x="7.62" y="27.94" smashed="yes">
+<attribute name="NAME" x="6.604" y="28.956" size="1.27" layer="25"/>
+<attribute name="VALUE" x="6.604" y="25.654" size="1.27" layer="27"/>
+</element>
+<element name="R4" library="adafruit" package="M0805" value="1k" x="12.7" y="27.94" smashed="yes">
+<attribute name="NAME" x="11.684" y="28.956" size="1.27" layer="25"/>
+<attribute name="VALUE" x="11.684" y="25.654" size="1.27" layer="27"/>
+</element>
+<element name="R5" library="adafruit" package="M0805" value="1k" x="17.78" y="27.94" smashed="yes">
+<attribute name="NAME" x="16.764" y="28.956" size="1.27" layer="25"/>
+<attribute name="VALUE" x="16.764" y="25.654" size="1.27" layer="27"/>
 </element>
 </elements>
@@
 <wire x1="13.716" y1="49.3776" x2="13.97" y2="49.53" width="0.6096" layer="1"/>
 <contactref element="R3" pad="2"/>
-<wire x1="3.49" y1="15.24" x2="6.4008" y2="46.6344" width="0" layer="19" extent="1-1"/>
+<wire x1="8.57" y1="27.94" x2="6.4008" y2="46.6344" width="0" layer="19" extent="1-1"/>
 </signal>
 <signal name="N$3">
@@
 <wire x1="11.43" y1="57.15" x2="13.97" y2="57.15" width="0.6096" layer="1"/>
 <contactref element="R2" pad="2"/>
-<wire x1="3.49" y1="21.59" x2="11.43" y2="57.15" width="0" layer="19" extent="1-1"/>
+<wire x1="8.57" y1="30.48" x2="11.43" y2="57.15" width="0" layer="19" extent="1-1"/>
 </signal>
 <signal name="N$4">
@@
 <wire x1="6.4008" y1="36.576" x2="6.35" y2="36.83" width="0.6096" layer="1"/>
 <contactref element="R5" pad="1"/>
-<wire x1="1.59" y1="2.54" x2="8.6868" y2="34.29" width="0" layer="19" extent="1-1"/>
+<wire x1="16.83" y1="27.94" x2="8.6868" y2="34.29" width="0" layer="19" extent="1-1"/>
 </signal>
 <signal name="N$10">
@@
 <wire x1="6.4008" y1="42.0624" x2="6.35" y2="41.91" width="0.6096" layer="1"/>
 <contactref element="R4" pad="1"/>
-<wire x1="1.59" y1="8.89" x2="6.35" y2="41.91" width="0" layer="19" extent="1-1"/>
+<wire x1="11.75" y1="27.94" x2="6.35" y2="41.91" width="0" layer="19" extent="1-1"/>
 </signal>
 <signal name="N$12">
@@
 <contactref element="RS232IN" pad="5"/>
 <contactref element="R3" pad="1"/>
-<wire x1="1.59" y1="15.24" x2="6.35" y2="46.99" width="0" layer="19" extent="1-1"/>
+<wire x1="6.67" y1="27.94" x2="6.35" y2="46.99" width="0" layer="19" extent="1-1"/>
 </signal>
 <signal name="N$11">
 <contactref element="RS232IN" pad="7"/>
 <contactref element="R2" pad="1"/>
-<wire x1="1.59" y1="21.59" x2="6.35" y2="52.07" width="0" layer="19" extent="1-1"/>
+<wire x1="6.67" y1="30.48" x2="6.35" y2="52.07" width="0" layer="19" extent="1-1"/>
 </signal>
 <signal name="N$15">
 <contactref element="RS485MODULE1" pad="J1.1"/>
 <contactref element="R5" pad="2"/>
-<wire x1="3.49" y1="2.54" x2="13.97" y2="34.29" width="0" layer="19" extent="1-1"/>
+<wire x1="18.73" y1="27.94" x2="13.97" y2="34.29" width="0" layer="19" extent="1-1"/>
 </signal>
 <signal name="N$14">
 <contactref element="RS485MODULE1" pad="J1.4"/>
 <contactref element="R4" pad="2"/>
-<wire x1="3.49" y1="8.89" x2="13.97" y2="41.91" width="0" layer="19" extent="1-1"/>
+<wire x1="13.65" y1="27.94" x2="13.97" y2="41.91" width="0" layer="19" extent="1-1"/>
 </signal>
 </signals>

Commit message: updated board
Parts:
- removed RS485OUT1, RS485OUT2: JST-XH-02-PIN-LONG-PAD, Rembrandt Electronics - JST XH Connectors v1-0:JST-XH-02-PACKAGE-LONG-PAD
- added RS485CONNECTEDTOD-D+GND, RS485OUTCONNECTEDTOD-D+GND: JST-XH-03-PIN-LONG-PAD, Rembrandt Electronics - JST XH Connectors v1-0:JST-XH-03-PACKAGE-LONG-PAD
Connections:
- net GND: now also RS485CONNECTEDTOD-D+GND.3, RS485OUTCONNECTEDTOD-D+GND.3
- net N$12: now also RS485CONNECTEDTOD-D+GND.1; no longer RS485OUT1.1
- net N$13: now also RS485CONNECTEDTOD-D+GND.2; no longer RS485OUT1.2
- net N$4: now also RS485OUTCONNECTEDTOD-D+GND.1; no longer RS485OUT2.1
- net N$6: now also RS485OUTCONNECTEDTOD-D+GND.2; no longer RS485OUT2.2
Routing:
- net N$12: track 29.2 -> 0.00 mm
Changed lines of the file:
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@@
 <attribute name="VALUE" x="12.954" y="59.944" size="1.27" layer="27"/>
-</element>
-<element name="RS485OUT1" library="Rembrandt Electronics - JST XH Connectors v1-0" package="JST-XH-02-PACKAGE-LONG-PAD" value="JST-XH-02-PIN-LONG-PAD" x="50.8" y="64.77" smashed="yes">
-<attribute name="NAME" x="55.38" y="69.405" size="1.016" layer="25" ratio="10" rot="R180"/>
-<attribute name="VALUE" x="47.4975" y="68.6625" size="1.016" layer="27" ratio="10"/>
-</element>
-<element name="RS485OUT2" library="Rembrandt Electronics - JST XH Connectors v1-0" package="JST-XH-02-PACKAGE-LONG-PAD" value="JST-XH-02-PIN-LONG-PAD" x="41.91" y="64.77" smashed="yes">
-<attribute name="NAME" x="45.22" y="69.405" size="1.016" layer="25" ratio="10" rot="R180"/>
-<attribute name="VALUE" x="38.6075" y="68.6625" size="1.016" layer="27" ratio="10"/>
 </element>
 <element name="RS232IN" library="Rembrandt Electronics - JST XH Connectors v1-0" package="JST-XH-07-PACKAGE-LONG-PAD" value="JST-XH-07-PIN-LONG-PAD" x="6.35" y="44.45" smashed="yes" rot="R90">
@@
 <attribute name="NAME" x="16.764" y="28.956" size="1.27" layer="25"/>
 <attribute name="VALUE" x="16.764" y="25.654" size="1.27" layer="27"/>
+</element>
+<element name="RS485OUTCONNECTEDTOD-D+GND" library="Rembrandt Electronics - JST XH Connectors v1-0" package="JST-XH-03-PACKAGE-LONG-PAD" value="JST-XH-03-PIN-LONG-PAD" x="7.62" y="19.05" smashed="yes">
+<attribute name="NAME" x="2.065" y="17.01" size="1.016" layer="25" ratio="10" rot="R90"/>
+<attribute name="VALUE" x="3.0175" y="22.9425" size="1.016" layer="27" ratio="10"/>
+</element>
+<element name="RS485CONNECTEDTOD-D+GND" library="Rembrandt Electronics - JST XH Connectors v1-0" package="JST-XH-03-PACKAGE-LONG-PAD" value="JST-XH-03-PIN-LONG-PAD" x="7.62" y="10.16" smashed="yes">
+<attribute name="NAME" x="2.065" y="8.12" size="1.016" layer="25" ratio="10" rot="R90"/>
+<attribute name="VALUE" x="3.0175" y="14.0525" size="1.016" layer="27" ratio="10"/>
 </element>
 </elements>
@@
 <wire x1="19.2024" y1="62.1792" x2="17.8308" y2="60.8076" width="0.6096" layer="1"/>
 <wire x1="19.2024" y1="62.1792" x2="19.27" y2="62.23" width="0.6096" layer="1"/>
+<contactref element="RS485CONNECTEDTOD-D+GND" pad="3"/>
+<contactref element="RS485OUTCONNECTEDTOD-D+GND" pad="3"/>
+<wire x1="10.16" y1="19.05" x2="6.35" y2="44.45" width="0" layer="19" extent="1-1"/>
+<wire x1="10.16" y1="10.16" x2="10.16" y2="19.05" width="0" layer="19" extent="1-1"/>
 </signal>
 <signal name="N$9">
@@
 <signal name="N$4">
 <contactref element="RS485MODULE2" pad="J2.2"/>
-<contactref element="RS485OUT2" pad="1"/>
 <wire x1="50.292" y1="54.864" x2="54.4068" y2="54.864" width="0.6096" layer="16"/>
 <wire x1="40.6908" y1="64.4652" x2="50.292" y2="54.864" width="0.6096" layer="16"/>
 <wire x1="54.4068" y1="54.864" x2="54.61" y2="54.61" width="0.6096" layer="16"/>
-<wire x1="40.6908" y1="64.4652" x2="40.64" y2="64.77" width="0.6096" layer="16"/>
+<contactref element="RS485OUTCONNECTEDTOD-D+GND" pad="1"/>
+<wire x1="5.08" y1="19.05" x2="40.6908" y2="64.4652" width="0" layer="19" extent="16-16"/>
 </signal>
 <signal name="N$6">
 <contactref element="RS485MODULE2" pad="J2.3"/>
-<contactref element="RS485OUT2" pad="2"/>
 <wire x1="43.434" y1="63.0936" x2="54.4068" y2="52.1208" width="0.6096" layer="1"/>
 <wire x1="43.434" y1="64.4652" x2="43.434" y2="63.0936" width="0.6096" layer="1"/>
 <wire x1="54.4068" y1="52.1208" x2="54.61" y2="52.07" width="0.6096" layer="1"/>
-<wire x1="43.434" y1="64.4652" x2="43.18" y2="64.77" width="0.6096" layer="1"/>
+<contactref element="RS485OUTCONNECTEDTOD-D+GND" pad="2"/>
+<wire x1="7.62" y1="19.05" x2="54.61" y2="52.07" width="0" layer="19" extent="1-1"/>
 </signal>
 <signal name="N$7">
@@
 </signal>
 <signal name="N$12">
+<contactref element="RS485CONNECTEDTOD-D+GND" pad="1"/>
 <contactref element="RS485MODULE1" pad="J2.2"/>
-<contactref element="RS485OUT1" pad="1"/>
-<wire x1="56.2356" y1="41.148" x2="54.864" y2="39.7764" width="0.6096" layer="1"/>
-<wire x1="56.2356" y1="58.0644" x2="56.2356" y2="41.148" width="0.6096" layer="1"/>
-<wire x1="51.6636" y1="62.6364" x2="56.2356" y2="58.0644" width="0.6096" layer="1"/>
-<wire x1="51.2064" y1="62.6364" x2="51.6636" y2="62.6364" width="0.6096" layer="1"/>
-<wire x1="49.3776" y1="64.4652" x2="51.2064" y2="62.6364" width="0.6096" layer="1"/>
-<wire x1="54.864" y1="39.7764" x2="54.61" y2="39.37" width="0.6096" layer="1"/>
-<wire x1="49.3776" y1="64.4652" x2="49.53" y2="64.77" width="0.6096" layer="1"/>
+<wire x1="5.08" y1="10.16" x2="54.61" y2="39.37" width="0" layer="19" extent="1-1"/>
 </signal>
 <signal name="N$13">
 <contactref element="RS485MODULE1" pad="J2.3"/>
-<contactref element="RS485OUT1" pad="2"/>
 <wire x1="57.15" y1="39.3192" x2="54.864" y2="37.0332" width="0.6096" layer="1"/>
 <wire x1="57.15" y1="59.436" x2="57.15" y2="39.3192" width="0.6096" layer="1"/>
 <wire x1="52.1208" y1="64.4652" x2="57.15" y2="59.436" width="0.6096" layer="1"/>
 <wire x1="54.864" y1="37.0332" x2="54.61" y2="36.83" width="0.6096" layer="1"/>
-<wire x1="52.1208" y1="64.4652" x2="52.07" y2="64.77" width="0.6096" layer="1"/>
+<contactref element="RS485CONNECTEDTOD-D+GND" pad="2"/>
+<wire x1="7.62" y1="10.16" x2="54.61" y2="36.83" width="0" layer="19" extent="1-1"/>
 </signal>
 <signal name="N$5">

Commit message: board updated
Parts:
- moved RS485CONNECTEDTOD-D+GND 70.6 mm to (50.8, 66.0)
- moved RS485OUTCONNECTEDTOD-D+GND 56.7 mm to (39.4, 66.0)
- moved 5V 1.27 mm to (29.2, 66.0)
Routing:
- net GND: track 108.9 -> 144.0 mm
- net N$12: track 0.00 -> 31.1 mm
- net N$3: track 2.54 -> 29.0 mm, vias 0 -> 1
- net N$11: track 0.00 -> 23.9 mm, vias 0 -> 1
- net N$5: track 0.00 -> 21.4 mm, vias 0 -> 1
- net N$14: track 0.00 -> 15.4 mm, vias 0 -> 1
- net N$2: track 8.75 -> 24.1 mm, vias 0 -> 1
- net N$10: track 7.48 -> 20.2 mm, vias 0 -> 1
- net N$4: track 18.0 -> 30.3 mm
- net N$8: track 3.49 -> 15.3 mm
- net N$15: track 0.00 -> 8.45 mm
- net N$6: track 17.1 -> 22.4 mm
- net N$7: track 7.65 -> 10.4 mm
- net N$1: track 9.88 -> 12.7 mm
- net N$13: track 30.8 -> 33.0 mm
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Other:
- board size 59.4 x 47 mm -> 60.6 x 47 mm

Commit message: updated board
Routing:
- net N$6: track 22.4 -> 28.5 mm
Changed lines of the file:
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@@
 <drawing>
 <settings>
-<setting alwaysvectorfont="yes"/>
+<setting alwaysvectorfont="no"/>
 <setting verticaltext="up"/>
 </settings>
@@
 <signal name="N$6">
 <contactref element="RS485MODULE2" pad="J2.3"/>
-<wire x1="43.434" y1="63.0936" x2="54.4068" y2="52.1208" width="0.6096" layer="1"/>
-<wire x1="43.434" y1="64.4652" x2="43.434" y2="63.5508" width="0.6096" layer="1"/>
-<wire x1="43.434" y1="63.5508" x2="43.434" y2="63.0936" width="0.6096" layer="1"/>
-<wire x1="54.4068" y1="52.1208" x2="54.61" y2="52.07" width="0.6096" layer="1"/>
+<wire x1="39.37" y1="66.04" x2="39.37" y2="53.34" width="0.6096" layer="1"/>
 <contactref element="RS485OUTCONNECTEDTOD-D+GND" pad="2"/>
-<wire x1="39.7764" y1="65.3796" x2="39.7764" y2="65.8368" width="0.6096" layer="1"/>
-<wire x1="41.6052" y1="63.5508" x2="39.7764" y2="65.3796" width="0.6096" layer="1"/>
-<wire x1="43.434" y1="63.5508" x2="41.6052" y2="63.5508" width="0.6096" layer="1"/>
-<wire x1="39.7764" y1="65.8368" x2="39.37" y2="66.04" width="0.6096" layer="1"/>
+<wire x1="54.61" y1="52.07" x2="40.64" y2="52.07" width="0.6096" layer="1"/>
+<wire x1="40.64" y1="52.07" x2="39.37" y2="53.34" width="0.6096" layer="1"/>
 </signal>
 <signal name="N$7">

Commit message: updated something
Connections:
- new net N$16: IC2.1, J1.1
- net VCC: no longer IC2.1, J1.1
Changed lines of the file:
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@@
 <signals>
 <signal name="VCC">
-<contactref element="J1" pad="1"/>
 <contactref element="R1" pad="1"/>
-<contactref element="IC2" pad="1"/>
 <contactref element="IC2" pad="2"/>
 <contactref element="RS485MODULE2" pad="J2.1"/>
@@
 <wire x1="23.7744" y1="69.4944" x2="23.7744" y2="65.8368" width="0.6096" layer="1"/>
 <wire x1="23.7744" y1="65.8368" x2="23.7744" y2="65.3796" width="0.6096" layer="1"/>
-<wire x1="23.7744" y1="65.3796" x2="23.85" y2="65.03" width="0.6096" layer="1"/>
 <wire x1="23.7744" y1="69.4944" x2="23.85" y2="69.59" width="0.6096" layer="1"/>
 <wire x1="23.7744" y1="65.8368" x2="27.5336" y2="65.8368" width="0.6096" layer="1"/>
@@
 <wire x1="6.4008" y1="58.5216" x2="10.0584" y2="62.1792" width="0.6096" layer="1"/>
 <wire x1="14.1732" y1="62.1792" x2="14.29" y2="62.23" width="0.6096" layer="1"/>
-<wire x1="6.4008" y1="58.5216" x2="6.35" y2="58.42" width="0.6096" layer="1"/>
 <wire x1="20.574" y1="69.9516" x2="23.7744" y2="69.9516" width="0.6096" layer="1"/>
 <wire x1="19.6596" y1="70.866" x2="20.574" y2="69.9516" width="0.6096" layer="1"/>
@@
 <via x="13.716" y="31.0896" extent="1-16" drill="0.35"/>
 </signal>
+<signal name="N$16">
+<contactref element="IC2" pad="1"/>
+<contactref element="J1" pad="1"/>
+<wire x1="6.35" y1="58.42" x2="23.85" y2="65.03" width="0" layer="19" extent="1-1"/>
+</signal>
 </signals>

Commit message: board updated
Parts:
- added C1: 0.1uF, adafruit:C0805
- added C2: 0.22uF, adafruit:C0805
- J1: value 6V-12V -> 7V-9V
- moved J1 1.27 mm to (5.08, 58.4)
- moved RS232IN 1.27 mm to (5.08, 44.5)
- moved R4 1.15 mm to (13.8, 27.8)
- moved R1 0.51 mm to (15.7, 62.2)
- moved R5 0.40 mm to (18.2, 27.8)
- moved R2 0.25 mm to (7.87, 30.5)
- renumbered RS485CONNECTEDTOD-D+GND to DRIVERD-D+GND, RS485OUTCONNECTEDTOD-D+GND to D-D+GND
Connections:
- net GND: now also C1.2, C2.2
- net N$16: now also C2.1
- net VCC: now also C1.1
Routing:
- net N$16: track 0.00 -> 31.2 mm, vias 0 -> 1
- net GND: track 144.0 -> 156.7 mm
- net VCC: track 88.1 -> 82.6 mm
- net N$10: track 20.2 -> 23.4 mm
- net N$15: track 8.45 -> 10.9 mm
- net N$11: track 23.9 -> 25.3 mm
- net N$7: track 10.4 -> 11.7 mm
- net N$5: track 21.4 -> 22.6 mm
- net N$1: track 12.7 -> 13.7 mm
- net N$13: track 33.0 -> 34.0 mm
- net N$8: track 15.3 -> 16.1 mm
- net N$2: track 24.1 -> 24.6 mm
Other:
- board text added: "Designed & Manufacturd by Pinwheel Robotics 17/11/2021 FutureBot Wi-Fi Shield V1.0"
- board text added: "Documentation at www.pinwheel.in"
- board text added: "FutureBot"
- board text added: "PINWHEEL ROBOTICS"
- board text added: "Wi-Fi Shield V1.0"
- board text added: "care@pinwheel.in"
- board text added: "www.pinwheel.in"

Commit message: updated gerber and corrected few things
Routing:
- added copper zone on layer 1, net GND
- added copper zone on layer 16, net GND
Other:
- board text added: "Designed & Manufacturd by Pinwheel Robotics 17/11/2021 FutureBot Dual Max485Shield V1.0"
- board text added: "Dual Max485 Shield V1.0"
- board text removed: "Designed & Manufacturd by Pinwheel Robotics 17/11/2021 FutureBot Wi-Fi Shield V1.0"
- board text removed: "Wi-Fi Shield V1.0"
Changed lines of the file:
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@@
 <text x="49.53" y="30.48" size="1.4224" layer="25" rot="R180">PINWHEEL ROBOTICS</text>
 <text x="31.75" y="26.67" size="1.778" layer="25">www.pinwheel.in</text>
-<text x="17.78" y="53.34" size="1.778" layer="25">Wi-Fi Shield V1.0</text>
+<text x="17.78" y="53.34" size="1.778" layer="25">Dual Max485 Shield V1.0</text>
 <text x="17.78" y="55.88" size="1.778" layer="25">FutureBot</text>
 <text x="43.18" y="35.56" size="1.778" layer="26" rot="MR0">Designed &amp; Manufacturd by
 Pinwheel Robotics
 17/11/2021
-FutureBot Wi-Fi Shield V1.0
+FutureBot
+Dual Max485Shield V1.0
 </text>
 <text x="33.02" y="59.69" size="1.778" layer="26" rot="MR180">care@pinwheel.in
@@
 <wire x1="19.27" y1="62.23" x2="17.2634" y2="60.2234" width="0.6096" layer="1"/>
 <wire x1="17.2634" y1="60.2234" x2="17.2466" y2="60.2234" width="0.6096" layer="1"/>
+<polygon width="0.1524" layer="1" isolate="0.6096">
+<vertex x="0" y="72.39"/>
+<vertex x="60.96" y="72.39"/>
+<vertex x="60.96" y="25.4"/>
+<vertex x="0" y="25.4"/>
+</polygon>
+<polygon width="0.1524" layer="16" isolate="0.6096">
+<vertex x="0" y="72.39"/>
+<vertex x="60.96" y="72.39"/>
+<vertex x="60.96" y="25.4"/>
+<vertex x="0" y="25.4"/>
+</polygon>
 </signal>
 <signal name="N$9">
@@
 <contactref element="RS485MODULE2" pad="J1.4"/>
 <contactref element="R2" pad="2"/>
-<wire x1="8.6868" y1="32.4612" x2="8.636" y2="32.4104" width="0.6096" layer="1"/>
 <wire x1="8.6868" y1="34.7472" x2="8.6868" y2="32.4612" width="0.6096" layer="16"/>
 <wire x1="11.43" y1="37.4904" x2="8.6868" y2="34.7472" width="0.6096" layer="16"/>
