File: PCBs/DualMax485.brd (EAGLE design)
At the start: 60.6 x 47 mm, 16 parts, among them IC2 7805DT, J1 7V-9V

Commit message: updated
Other:
- board text added: "Designed & Manufacturd by Pinwheel Robotics 27/11/2021 FutureBot Dual MAX485 Shield V1.0"
- board text removed: "Designed & Manufacturd by Pinwheel Robotics 17/11/2021 FutureBot Dual Max485Shield V1.0"
Changed lines of the file:
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@@
 <text x="17.78" y="53.34" size="1.778" layer="25">Dual Max485 Shield V1.0</text>
 <text x="17.78" y="55.88" size="1.778" layer="25">FutureBot</text>
-<text x="43.18" y="35.56" size="1.778" layer="26" rot="MR0">Designed &amp; Manufacturd by
-Pinwheel Robotics
-17/11/2021
-FutureBot
-Dual Max485Shield V1.0
-</text>
 <text x="33.02" y="59.69" size="1.778" layer="26" rot="MR180">care@pinwheel.in
 </text>
 <text x="46.99" y="36.83" size="1.778" layer="26" rot="MR90">Documentation at
 www.pinwheel.in</text>
+<text x="45.72" y="35.56" size="1.778" layer="26" rot="MR0">Designed &amp; Manufacturd by
+Pinwheel Robotics
+27/11/2021
+FutureBot
+Dual MAX485 Shield V1.0
+</text>
 </plain>
 <attributes>
@@
 </element>
 <element name="RS485MODULE2" library="diy-modules" package="RS485-TTL-CONVERTER" value="RS485-TTL-CONVERTER" x="34.29" y="53.34" smashed="yes">
-<attribute name="NAME" x="34.29" y="50.165" size="1.27" layer="25" align="bottom-center"/>
+<attribute name="NAME" x="31.75" y="51.435" size="1.27" layer="25" align="bottom-center"/>
 <attribute name="VALUE" x="34.29" y="45.085" size="1.27" layer="27" align="top-center"/>
 </element>
