File: PCBs/NodeMCU.sch (EAGLE design)
At the start: 15 parts, among them IC1 7805DT

Commit message: updated board
Parts:
- added R2, R3: 1k, adafruit:R-US_M0805
Connections:
- new net N$10: R3.1, RS232RST-2.S
- new net N$5: R2.1, RS232RST-1.S
- net N$6: now also R2.2; no longer RS232RST-1.S
- net N$8: now also R3.2; no longer RS232RST-2.S
Changed lines of the file:
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@@
 <part name="5V" library="Rembrandt Electronics - JST XH Connectors v1-0" deviceset="JST-XH-02-PIN" device="-LONG-PAD"/>
 <part name="SUPPLY14" library="supply2" library_urn="urn:adsk.eagle:library:372" deviceset="GND" device=""/>
+<part name="R2" library="adafruit" deviceset="R-US_" device="M0805" value="1k"/>
+<part name="R3" library="adafruit" deviceset="R-US_" device="M0805" value="1k"/>
 </parts>
 <sheets>
@@
 <instance part="SUPPLY14" gate="GND" x="31.75" y="105.41" smashed="yes" rot="R180">
 <attribute name="VALUE" x="33.655" y="108.585" size="1.778" layer="96" rot="R180"/>
+</instance>
+<instance part="R2" gate="G$1" x="101.6" y="111.76" smashed="yes" rot="R180">
+<attribute name="NAME" x="100.33" y="115.3414" size="1.778" layer="95" rot="R180"/>
+<attribute name="VALUE" x="105.41" y="115.062" size="1.778" layer="96" rot="R180"/>
+</instance>
+<instance part="R3" gate="G$1" x="99.06" y="106.68" smashed="yes" rot="R180">
+<attribute name="NAME" x="102.87" y="105.1814" size="1.778" layer="95" rot="R180"/>
+<attribute name="VALUE" x="97.79" y="104.902" size="1.778" layer="96" rot="R180"/>
 </instance>
 </instances>
@@
 <pinref part="U$2" gate="G$1" pin="24"/>
 <wire x1="71.12" y1="99.06" x2="71.12" y2="71.12" width="0.1524" layer="91"/>
-<wire x1="81.28" y1="99.06" x2="81.28" y2="104.14" width="0.1524" layer="91"/>
 <wire x1="87.63" y1="71.12" x2="71.12" y2="71.12" width="0.1524" layer="91"/>
-<pinref part="RS232RST" gate="-1" pin="S"/>
-<wire x1="116.84" y1="111.76" x2="109.22" y2="111.76" width="0.1524" layer="91"/>
-<wire x1="109.22" y1="111.76" x2="109.22" y2="104.14" width="0.1524" layer="91"/>
-<wire x1="109.22" y1="104.14" x2="81.28" y2="104.14" width="0.1524" layer="91"/>
+<wire x1="81.28" y1="99.06" x2="81.28" y2="111.76" width="0.1524" layer="91"/>
+<pinref part="R2" gate="G$1" pin="2"/>
+<wire x1="81.28" y1="111.76" x2="96.52" y2="111.76" width="0.1524" layer="91"/>
 </segment>
 </net>
@@
 <wire x1="73.66" y1="68.58" x2="87.63" y2="68.58" width="0.1524" layer="91"/>
 <pinref part="U$2" gate="G$1" pin="23"/>
-<pinref part="RS232RST" gate="-2" pin="S"/>
-<wire x1="83.82" y1="101.6" x2="83.82" y2="96.52" width="0.1524" layer="91"/>
-<wire x1="116.84" y1="109.22" x2="111.76" y2="109.22" width="0.1524" layer="91"/>
-<wire x1="111.76" y1="109.22" x2="111.76" y2="101.6" width="0.1524" layer="91"/>
-<wire x1="111.76" y1="101.6" x2="83.82" y2="101.6" width="0.1524" layer="91"/>
+<wire x1="83.82" y1="96.52" x2="83.82" y2="106.68" width="0.1524" layer="91"/>
+<pinref part="R3" gate="G$1" pin="2"/>
+<wire x1="83.82" y1="106.68" x2="93.98" y2="106.68" width="0.1524" layer="91"/>
 </segment>
 </net>
@@
 </segment>
 </net>
+<net name="N$5" class="0">
+<segment>
+<pinref part="RS232RST" gate="-1" pin="S"/>
+<wire x1="116.84" y1="111.76" x2="106.68" y2="111.76" width="0.1524" layer="91"/>
+<pinref part="R2" gate="G$1" pin="1"/>
+</segment>
+</net>
+<net name="N$10" class="0">
+<segment>
+<pinref part="RS232RST" gate="-2" pin="S"/>
+<wire x1="116.84" y1="109.22" x2="111.76" y2="109.22" width="0.1524" layer="91"/>
+<wire x1="111.76" y1="109.22" x2="111.76" y2="106.68" width="0.1524" layer="91"/>
+<pinref part="R3" gate="G$1" pin="1"/>
+<wire x1="104.14" y1="106.68" x2="111.76" y2="106.68" width="0.1524" layer="91"/>
+</segment>
+</net>

Commit message: Changed Pin number in future if we connect LCD module to it.
Parts:
- 6V-12V: value 6V-12V -> 7V-9V
Connections:
- removed net N$14: LCD-PCF8574-1.S, U$2.29
- removed net N$15: LCD-PCF8574-2.S, U$2.28
- new net N$12: GPIO-2.S, R4.2, U$2.25
- new net N$13: GPIO-1.S, R5.2, U$2.20
- net N$2: now also LCD-PCF8574-2.S, U$2.18; no longer GPIO-1.S, R5.2, U$2.17
- net N$7: now also LCD-PCF8574-1.S, U$2.17; no longer GPIO-2.S, R4.2, U$2.18
Changed lines of the file:
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@@
 <part name="SUPPLY6" library="supply2" library_urn="urn:adsk.eagle:library:372" deviceset="VCC" device=""/>
 <part name="SUPPLY7" library="supply2" library_urn="urn:adsk.eagle:library:372" deviceset="GND" device=""/>
-<part name="6V-12V" library="SparkFun-Connectors" library_urn="urn:adsk.eagle:library:513" deviceset="CONN_02" device="5MM" package3d_urn="urn:adsk.eagle:package:38044/1" value="6V-12V"/>
+<part name="6V-12V" library="SparkFun-Connectors" library_urn="urn:adsk.eagle:library:513" deviceset="CONN_02" device="5MM" package3d_urn="urn:adsk.eagle:package:38044/1" value="7V-9V"/>
 <part name="SUPPLY8" library="supply2" library_urn="urn:adsk.eagle:library:372" deviceset="GND" device=""/>
 <part name="SUPPLY9" library="supply2" library_urn="urn:adsk.eagle:library:372" deviceset="GND" device=""/>
@@
 <net name="N$2" class="0">
 <segment>
+<wire x1="96.52" y1="55.88" x2="96.52" y2="78.74" width="0.1524" layer="91"/>
+<wire x1="96.52" y1="78.74" x2="91.44" y2="78.74" width="0.1524" layer="91"/>
+<wire x1="91.44" y1="78.74" x2="91.44" y2="101.6" width="0.1524" layer="91"/>
+<wire x1="91.44" y1="101.6" x2="88.9" y2="101.6" width="0.1524" layer="91"/>
+<wire x1="88.9" y1="101.6" x2="88.9" y2="109.22" width="0.1524" layer="91"/>
+<wire x1="88.9" y1="109.22" x2="96.52" y2="109.22" width="0.1524" layer="91"/>
+<pinref part="LCD-PCF8574" gate="-2" pin="S"/>
+<wire x1="76.2" y1="116.84" x2="96.52" y2="116.84" width="0.1524" layer="91"/>
+<wire x1="96.52" y1="109.22" x2="96.52" y2="116.84" width="0.1524" layer="91"/>
+<pinref part="U$2" gate="G$1" pin="18"/>
+<wire x1="87.63" y1="55.88" x2="96.52" y2="55.88" width="0.1524" layer="91"/>
+</segment>
+</net>
+<net name="N$7" class="0">
+<segment>
+<pinref part="LCD-PCF8574" gate="-1" pin="S"/>
+<wire x1="76.2" y1="114.3" x2="93.98" y2="114.3" width="0.1524" layer="91"/>
 <pinref part="U$2" gate="G$1" pin="17"/>
-<pinref part="R5" gate="G$1" pin="2"/>
-<wire x1="87.63" y1="53.34" x2="73.66" y2="53.34" width="0.1524" layer="91"/>
-<wire x1="73.66" y1="53.34" x2="73.66" y2="60.96" width="0.1524" layer="91"/>
-<junction x="73.66" y="53.34"/>
-<pinref part="GPIO" gate="-1" pin="S"/>
-<wire x1="73.66" y1="60.96" x2="35.56" y2="60.96" width="0.1524" layer="91"/>
-<wire x1="35.56" y1="60.96" x2="35.56" y2="63.5" width="0.1524" layer="91"/>
-</segment>
-</net>
-<net name="N$7" class="0">
-<segment>
-<pinref part="U$2" gate="G$1" pin="18"/>
-<pinref part="R4" gate="G$1" pin="2"/>
-<wire x1="87.63" y1="55.88" x2="71.12" y2="55.88" width="0.1524" layer="91"/>
-<pinref part="GPIO" gate="-2" pin="S"/>
-<wire x1="71.12" y1="55.88" x2="71.12" y2="66.04" width="0.1524" layer="91"/>
-<wire x1="71.12" y1="66.04" x2="35.56" y2="66.04" width="0.1524" layer="91"/>
-<junction x="71.12" y="55.88"/>
-</segment>
-</net>
-<net name="N$14" class="0">
-<segment>
-<pinref part="U$2" gate="G$1" pin="29"/>
-<wire x1="87.63" y1="83.82" x2="88.9" y2="83.82" width="0.1524" layer="91"/>
-<wire x1="88.9" y1="83.82" x2="88.9" y2="114.3" width="0.1524" layer="91"/>
-<pinref part="LCD-PCF8574" gate="-1" pin="S"/>
-<wire x1="88.9" y1="114.3" x2="76.2" y2="114.3" width="0.1524" layer="91"/>
-</segment>
-</net>
-<net name="N$15" class="0">
-<segment>
-<pinref part="U$2" gate="G$1" pin="28"/>
-<wire x1="87.63" y1="81.28" x2="91.44" y2="81.28" width="0.1524" layer="91"/>
-<wire x1="91.44" y1="81.28" x2="91.44" y2="116.84" width="0.1524" layer="91"/>
-<pinref part="LCD-PCF8574" gate="-2" pin="S"/>
-<wire x1="91.44" y1="116.84" x2="76.2" y2="116.84" width="0.1524" layer="91"/>
+<wire x1="87.63" y1="53.34" x2="93.98" y2="53.34" width="0.1524" layer="91"/>
+<wire x1="93.98" y1="53.34" x2="93.98" y2="114.3" width="0.1524" layer="91"/>
 </segment>
 </net>
@@
 </segment>
 </net>
+<net name="N$12" class="0">
+<segment>
+<pinref part="GPIO" gate="-2" pin="S"/>
+<pinref part="R4" gate="G$1" pin="2"/>
+<wire x1="71.12" y1="55.88" x2="71.12" y2="66.04" width="0.1524" layer="91"/>
+<wire x1="71.12" y1="66.04" x2="35.56" y2="66.04" width="0.1524" layer="91"/>
+<pinref part="U$2" gate="G$1" pin="25"/>
+<wire x1="87.63" y1="73.66" x2="76.2" y2="73.66" width="0.1524" layer="91"/>
+<wire x1="76.2" y1="73.66" x2="76.2" y2="66.04" width="0.1524" layer="91"/>
+<wire x1="76.2" y1="66.04" x2="71.12" y2="66.04" width="0.1524" layer="91"/>
+<junction x="71.12" y="66.04"/>
+</segment>
+</net>
+<net name="N$13" class="0">
+<segment>
+<pinref part="GPIO" gate="-1" pin="S"/>
+<pinref part="R5" gate="G$1" pin="2"/>
+<wire x1="73.66" y1="53.34" x2="73.66" y2="60.96" width="0.1524" layer="91"/>
+<wire x1="73.66" y1="60.96" x2="35.56" y2="60.96" width="0.1524" layer="91"/>
+<wire x1="35.56" y1="60.96" x2="35.56" y2="63.5" width="0.1524" layer="91"/>
+<pinref part="U$2" gate="G$1" pin="20"/>
+<wire x1="87.63" y1="60.96" x2="73.66" y2="60.96" width="0.1524" layer="91"/>
+<junction x="73.66" y="60.96"/>
+</segment>
+</net>

Commit message: updated
Parts:
- renumbered 6V-12V to POWER
Changed lines of the file:
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@@
 <part name="SUPPLY6" library="supply2" library_urn="urn:adsk.eagle:library:372" deviceset="VCC" device=""/>
 <part name="SUPPLY7" library="supply2" library_urn="urn:adsk.eagle:library:372" deviceset="GND" device=""/>
-<part name="6V-12V" library="SparkFun-Connectors" library_urn="urn:adsk.eagle:library:513" deviceset="CONN_02" device="5MM" package3d_urn="urn:adsk.eagle:package:38044/1" value="7V-9V"/>
+<part name="POWER" library="SparkFun-Connectors" library_urn="urn:adsk.eagle:library:513" deviceset="CONN_02" device="5MM" package3d_urn="urn:adsk.eagle:package:38044/1" value="7V-9V"/>
 <part name="SUPPLY8" library="supply2" library_urn="urn:adsk.eagle:library:372" deviceset="GND" device=""/>
 <part name="SUPPLY9" library="supply2" library_urn="urn:adsk.eagle:library:372" deviceset="GND" device=""/>
@@
 <attribute name="VALUE" x="114.935" y="76.835" size="1.778" layer="96"/>
 </instance>
-<instance part="6V-12V" gate="G$1" x="45.72" y="116.84" smashed="yes" rot="R270">
+<instance part="POWER" gate="G$1" x="45.72" y="116.84" smashed="yes" rot="R270">
 <attribute name="VALUE" x="40.894" y="119.38" size="1.778" layer="96" font="vector" rot="R270"/>
 <attribute name="NAME" x="43.18" y="119.888" size="1.778" layer="95" font="vector"/>
@@
 <segment>
 <pinref part="SUPPLY8" gate="GND" pin="GND"/>
-<pinref part="6V-12V" gate="G$1" pin="2"/>
+<pinref part="POWER" gate="G$1" pin="2"/>
 <wire x1="48.26" y1="107.95" x2="48.26" y2="109.22" width="0.1524" layer="91"/>
 </segment>
@@
 <net name="N$9" class="0">
 <segment>
-<pinref part="6V-12V" gate="G$1" pin="1"/>
+<pinref part="POWER" gate="G$1" pin="1"/>
 <wire x1="45.72" y1="109.22" x2="38.1" y2="109.22" width="0.1524" layer="91"/>
 <wire x1="38.1" y1="109.22" x2="38.1" y2="99.06" width="0.1524" layer="91"/>
