File: PCBs/NodeMCU.brd (EAGLE design)
At the start: 59.4 x 53.3 mm, 15 parts, among them IC1 7805DT

Commit message: updated board
Parts:
- added R2, R3: 1k, adafruit:M0805
Connections:
- new net N$10: R3.1, RS232RST.2
- new net N$5: R2.1, RS232RST.1
- net N$6: now also R2.2; no longer RS232RST.1
- net N$8: now also R3.2; no longer RS232RST.2
Routing:
- net VCC: track 121.5 -> 130.1 mm
- net N$5: track 0.00 -> 7.81 mm
- net N$10: track 0.00 -> 5.61 mm
- net N$6: track 17.4 -> 13.0 mm
- net N$8: track 17.4 -> 15.5 mm
- net N$11: track 57.8 -> 59.6 mm
- net N$2: track 65.5 -> 66.9 mm
- net GND: track 270.3 -> 271.0 mm
- net N$9: track 23.6 -> 24.2 mm

Commit message: Changed Pin number in future if we connect LCD module to it.
Parts:
- 6V-12V: value 6V-12V -> 7V-9V
Connections:
- removed net N$14: LCD-PCF8574.1, U$2.29
- removed net N$15: LCD-PCF8574.2, U$2.28
- new net N$12: GPIO.2, R4.2, U$2.25
- new net N$13: GPIO.1, R5.2, U$2.20
- net N$2: now also LCD-PCF8574.2, U$2.18; no longer GPIO.1, R5.2, U$2.17
- net N$7: now also LCD-PCF8574.1, U$2.17; no longer GPIO.2, R4.2, U$2.18
Routing:
- net N$13: track 0.00 -> 48.9 mm
- net N$2: track 66.9 -> 21.4 mm
- net N$7: track 65.3 -> 29.3 mm
- net N$12: track 0.00 -> 32.5 mm
- net N$15: track 17.0 -> 0.00 mm
- net N$14: track 16.8 -> 0.00 mm
- added copper zone on layer 1, net GND
- added copper zone on layer 16, net GND
Changed lines of the file:
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@@
 <drawing>
 <settings>
-<setting alwaysvectorfont="no"/>
+<setting alwaysvectorfont="yes"/>
 <setting verticaltext="up"/>
 </settings>
@@
 <elements>
 <element name="U$2" library="NODEMCU" package="NODEMCUESP8266" value="NodeMCU-ESP12E" x="59.69" y="24.13" smashed="yes" rot="R180"/>
-<element name="6V-12V" library="SparkFun-Connectors" library_urn="urn:adsk.eagle:library:513" package="SCREWTERMINAL-5MM-2" package3d_urn="urn:adsk.eagle:package:38044/1" value="6V-12V" x="34.29" y="13.97" smashed="yes" rot="R270">
+<element name="6V-12V" library="SparkFun-Connectors" library_urn="urn:adsk.eagle:library:513" package="SCREWTERMINAL-5MM-2" package3d_urn="urn:adsk.eagle:package:38044/1" value="7V-9V" x="34.29" y="13.97" smashed="yes" rot="R270">
 <attribute name="NAME" x="29.718" y="13.208" size="1.27" layer="25" font="vector" ratio="12" rot="R270"/>
 <attribute name="SF_SKU" value="PRT-08432" x="34.29" y="13.97" size="1.778" layer="27" rot="R270" display="off"/>
@@
 <wire x1="37.608" y1="33.528" x2="39.624" y2="33.528" width="0.4572" layer="1"/>
 <wire x1="39.624" y1="33.528" x2="40.64" y2="34.544" width="0.4572" layer="1"/>
+<polygon width="0.4572" layer="1" isolate="0.8128">
+<vertex x="26.416" y="53.848"/>
+<vertex x="86.36" y="53.848"/>
+<vertex x="86.36" y="0"/>
+<vertex x="26.416" y="0"/>
+</polygon>
+<polygon width="0.4572" layer="16" isolate="0.8128">
+<vertex x="26.416" y="53.848"/>
+<vertex x="86.36" y="53.848"/>
+<vertex x="86.36" y="0"/>
+<vertex x="26.416" y="0"/>
+</polygon>
 </signal>
 <signal name="VCC">
@@
 </signal>
 <signal name="N$2">
+<contactref element="LCD-PCF8574" pad="2"/>
+<contactref element="U$2" pad="18"/>
+<wire x1="71.247" y1="39.243" x2="70.104" y2="39.243" width="0.4572" layer="16"/>
+<wire x1="80.01" y1="30.48" x2="71.247" y2="39.243" width="0.4572" layer="16"/>
+<wire x1="80.01" y1="26.289" x2="80.01" y2="30.48" width="0.4572" layer="16"/>
+<wire x1="82.296" y1="24.003" x2="80.01" y2="26.289" width="0.4572" layer="16"/>
+<wire x1="70.104" y1="39.243" x2="69.85" y2="39.37" width="0.4572" layer="16"/>
+<wire x1="82.296" y1="24.003" x2="82.296" y2="24.13" width="0.4572" layer="16"/>
+</signal>
+<signal name="N$7">
+<contactref element="LCD-PCF8574" pad="1"/>
 <contactref element="U$2" pad="17"/>
-<contactref element="R5" pad="2"/>
-<contactref element="GPIO" pad="1"/>
-<wire x1="66.04" y1="39.243" x2="68.707" y2="41.91" width="0.4572" layer="16"/>
-<wire x1="66.04" y1="9.017" x2="66.04" y2="39.243" width="0.4572" layer="16"/>
-<wire x1="68.199" y1="6.858" x2="66.04" y2="9.017" width="0.4572" layer="16"/>
-<wire x1="78.486" y1="6.858" x2="68.199" y2="6.858" width="0.4572" layer="16"/>
-<wire x1="82.296" y1="10.668" x2="78.486" y2="6.858" width="0.4572" layer="16"/>
-<wire x1="68.707" y1="41.91" x2="69.85" y2="41.91" width="0.4572" layer="16"/>
-<wire x1="82.296" y1="10.668" x2="81.0514" y2="11.9126" width="0.4572" layer="1"/>
-<wire x1="81.0514" y1="11.9126" x2="80.997425" y2="11.9126" width="0.4572" layer="1"/>
-<wire x1="80.997425" y1="11.9126" x2="79.248" y2="13.662025" width="0.4572" layer="1"/>
-<wire x1="79.248" y1="13.662025" x2="79.248" y2="20.32" width="0.4572" layer="1"/>
-<wire x1="79.248" y1="20.32" x2="77.15" y2="20.32" width="0.4572" layer="1"/>
-</signal>
-<signal name="N$7">
-<contactref element="U$2" pad="18"/>
+<wire x1="67.818" y1="40.005" x2="69.723" y2="41.91" width="0.4572" layer="16"/>
+<wire x1="67.818" y1="38.862" x2="67.818" y2="40.005" width="0.4572" layer="16"/>
+<wire x1="68.58" y1="38.1" x2="67.818" y2="38.862" width="0.4572" layer="16"/>
+<wire x1="71.247" y1="38.1" x2="68.58" y2="38.1" width="0.4572" layer="16"/>
+<wire x1="79.248" y1="30.099" x2="71.247" y2="38.1" width="0.4572" layer="16"/>
+<wire x1="79.248" y1="24.384" x2="79.248" y2="30.099" width="0.4572" layer="16"/>
+<wire x1="82.296" y1="21.336" x2="79.248" y2="24.384" width="0.4572" layer="16"/>
+<wire x1="69.723" y1="41.91" x2="69.85" y2="41.91" width="0.4572" layer="16"/>
+<wire x1="82.296" y1="21.336" x2="82.296" y2="21.59" width="0.4572" layer="16"/>
+</signal>
+<signal name="N$5">
+<contactref element="RS232RST" pad="1"/>
+<contactref element="R2" pad="1"/>
+<wire x1="82.55" y1="35.56" x2="78.232" y2="35.56" width="0.4572" layer="1"/>
+<wire x1="78.232" y1="35.56" x2="77.15" y2="34.478" width="0.4572" layer="1"/>
+<wire x1="77.15" y1="34.478" x2="77.15" y2="32.512" width="0.4572" layer="1"/>
+</signal>
+<signal name="N$10">
+<contactref element="RS232RST" pad="2"/>
+<contactref element="R3" pad="1"/>
+<wire x1="77.15" y1="37.592" x2="78.232" y2="37.592" width="0.4572" layer="1"/>
+<wire x1="78.232" y1="37.592" x2="78.74" y2="38.1" width="0.4572" layer="1"/>
+<wire x1="78.74" y1="38.1" x2="82.55" y2="38.1" width="0.4572" layer="1"/>
+</signal>
+<signal name="N$12">
 <contactref element="R4" pad="2"/>
 <contactref element="GPIO" pad="2"/>
-<wire x1="67.818" y1="37.338" x2="69.85" y2="39.37" width="0.4572" layer="16"/>
-<wire x1="67.818" y1="8.382" x2="67.818" y2="37.338" width="0.4572" layer="16"/>
-<wire x1="68.58" y1="7.62" x2="67.818" y2="8.382" width="0.4572" layer="16"/>
-<wire x1="76.581" y1="7.62" x2="68.58" y2="7.62" width="0.4572" layer="16"/>
-<wire x1="82.296" y1="13.335" x2="76.581" y2="7.62" width="0.4572" layer="16"/>
-<wire x1="82.296" y1="13.335" x2="82.296" y2="13.208" width="0.4572" layer="16"/>
 <wire x1="77.15" y1="5.08" x2="81.42860625" y2="5.08" width="0.4572" layer="1"/>
 <wire x1="81.42860625" y1="5.08" x2="82.16520625" y2="5.8166" width="0.4572" layer="1"/>
@@
 <wire x1="84.7854" y1="12.192" x2="84.7854" y2="7.5694" width="0.4572" layer="1"/>
 <wire x1="84.7854" y1="7.5694" x2="83.0326" y2="5.8166" width="0.4572" layer="1"/>
-</signal>
-<signal name="N$14">
-<contactref element="U$2" pad="29"/>
-<contactref element="LCD-PCF8574" pad="1"/>
-<wire x1="72.39" y1="11.43" x2="69.85" y2="11.43" width="0.4572" layer="16"/>
-<wire x1="82.296" y1="21.336" x2="72.39" y2="11.43" width="0.4572" layer="16"/>
-<wire x1="82.296" y1="21.336" x2="82.296" y2="21.59" width="0.4572" layer="16"/>
-</signal>
-<signal name="N$15">
-<contactref element="U$2" pad="28"/>
-<contactref element="LCD-PCF8574" pad="2"/>
-<wire x1="72.009" y1="14.097" x2="70.104" y2="14.097" width="0.4572" layer="16"/>
-<wire x1="82.296" y1="24.384" x2="72.009" y2="14.097" width="0.4572" layer="16"/>
-<wire x1="70.104" y1="14.097" x2="69.85" y2="13.97" width="0.4572" layer="16"/>
-<wire x1="82.296" y1="24.384" x2="82.296" y2="24.13" width="0.4572" layer="16"/>
-</signal>
-<signal name="N$5">
-<contactref element="RS232RST" pad="1"/>
-<contactref element="R2" pad="1"/>
-<wire x1="82.55" y1="35.56" x2="78.232" y2="35.56" width="0.4572" layer="1"/>
-<wire x1="78.232" y1="35.56" x2="77.15" y2="34.478" width="0.4572" layer="1"/>
-<wire x1="77.15" y1="34.478" x2="77.15" y2="32.512" width="0.4572" layer="1"/>
-</signal>
-<signal name="N$10">
-<contactref element="RS232RST" pad="2"/>
-<contactref element="R3" pad="1"/>
-<wire x1="77.15" y1="37.592" x2="78.232" y2="37.592" width="0.4572" layer="1"/>
-<wire x1="78.232" y1="37.592" x2="78.74" y2="38.1" width="0.4572" layer="1"/>
-<wire x1="78.74" y1="38.1" x2="82.55" y2="38.1" width="0.4572" layer="1"/>
+<contactref element="U$2" pad="25"/>
+<wire x1="73.914" y1="21.336" x2="70.104" y2="21.336" width="0.4572" layer="16"/>
+<wire x1="82.296" y1="12.954" x2="73.914" y2="21.336" width="0.4572" layer="16"/>
+<wire x1="70.104" y1="21.336" x2="69.85" y2="21.59" width="0.4572" layer="16"/>
+<wire x1="82.296" y1="12.954" x2="82.296" y2="13.208" width="0.4572" layer="16"/>
+</signal>
+<signal name="N$13">
+<contactref element="R5" pad="2"/>
+<contactref element="GPIO" pad="1"/>
+<wire x1="82.296" y1="10.668" x2="81.0514" y2="11.9126" width="0.4572" layer="1"/>
+<wire x1="81.0514" y1="11.9126" x2="80.997425" y2="11.9126" width="0.4572" layer="1"/>
+<wire x1="80.997425" y1="11.9126" x2="79.248" y2="13.662025" width="0.4572" layer="1"/>
+<wire x1="79.248" y1="13.662025" x2="79.248" y2="20.32" width="0.4572" layer="1"/>
+<wire x1="79.248" y1="20.32" x2="77.15" y2="20.32" width="0.4572" layer="1"/>
+<contactref element="U$2" pad="20"/>
+<wire x1="67.818" y1="32.385" x2="69.723" y2="34.29" width="0.4572" layer="16"/>
+<wire x1="67.818" y1="16.002" x2="67.818" y2="32.385" width="0.4572" layer="16"/>
+<wire x1="68.58" y1="15.24" x2="67.818" y2="16.002" width="0.4572" layer="16"/>
+<wire x1="77.343" y1="15.24" x2="68.58" y2="15.24" width="0.4572" layer="16"/>
+<wire x1="81.915" y1="10.668" x2="77.343" y2="15.24" width="0.4572" layer="16"/>
+<wire x1="82.296" y1="10.668" x2="81.915" y2="10.668" width="0.4572" layer="16"/>
+<wire x1="69.723" y1="34.29" x2="69.85" y2="34.29" width="0.4572" layer="16"/>
 </signal>
 </signals>

Commit message: updated
Parts:
- renumbered 6V-12V to POWER
Other:
- board text added: "Designed & Manufacturd by Pinwheel Robotics 17/11/2021 FutureBot Wi-Fi Shield V1.0"
- board text added: "Documentation at"
- board text added: "FutureBot Wi-Fi Shield V1.0"
- board text added: "PINWHEEL ROBOTICS www.pinwheel.in"
- board text added: "care@pinwheel.in"
Changed lines of the file:
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@@
 <layers>
 <layer number="1" name="Top" color="4" fill="1" visible="yes" active="yes"/>
-<layer number="16" name="Bottom" color="1" fill="1" visible="yes" active="yes"/>
+<layer number="16" name="Bottom" color="1" fill="1" visible="no" active="yes"/>
 <layer number="17" name="Pads" color="2" fill="1" visible="yes" active="yes"/>
 <layer number="18" name="Vias" color="2" fill="1" visible="yes" active="yes"/>
@@
 <hole x="83.312" y="3.048" drill="3.048"/>
 <hole x="29.464" y="3.048" drill="3.048"/>
+<text x="35.56" y="50.8" size="1.778" layer="25">PINWHEEL ROBOTICS www.pinwheel.in</text>
+<text x="50.8" y="2.032" size="1.778" layer="26" rot="MR90">Designed &amp; Manufacturd by
+Pinwheel Robotics
+17/11/2021
+FutureBot Wi-Fi Shield V1.0
+</text>
+<text x="27.432" y="5.08" size="1.778" layer="26" rot="MR90">Documentation at
+</text>
+<text x="68.072" y="44.704" size="1.778" layer="26" rot="MR0">care@pinwheel.in
+</text>
+<text x="46.736" y="39.624" size="1.778" layer="25">FutureBot
+Wi-Fi Shield V1.0
+</text>
 </plain>
 <attributes>
@@
 <elements>
 <element name="U$2" library="NODEMCU" package="NODEMCUESP8266" value="NodeMCU-ESP12E" x="59.69" y="24.13" smashed="yes" rot="R180"/>
-<element name="6V-12V" library="SparkFun-Connectors" library_urn="urn:adsk.eagle:library:513" package="SCREWTERMINAL-5MM-2" package3d_urn="urn:adsk.eagle:package:38044/1" value="7V-9V" x="34.29" y="13.97" smashed="yes" rot="R270">
+<element name="POWER" library="SparkFun-Connectors" library_urn="urn:adsk.eagle:library:513" package="SCREWTERMINAL-5MM-2" package3d_urn="urn:adsk.eagle:package:38044/1" value="7V-9V" x="34.29" y="13.97" smashed="yes" rot="R270">
 <attribute name="NAME" x="29.718" y="13.208" size="1.27" layer="25" font="vector" ratio="12" rot="R270"/>
 <attribute name="SF_SKU" value="PRT-08432" x="34.29" y="13.97" size="1.778" layer="27" rot="R270" display="off"/>
@@
 <signals>
 <signal name="GND">
-<contactref element="6V-12V" pad="2"/>
+<contactref element="POWER" pad="2"/>
 <contactref element="U$2" pad="2"/>
 <contactref element="RS232RST" pad="4"/>
@@
 </signal>
 <signal name="N$9">
-<contactref element="6V-12V" pad="1"/>
+<contactref element="POWER" pad="1"/>
 <contactref element="IC1" pad="1"/>
 <contactref element="C1" pad="1"/>
@@
 </drawing>
 <compatibility>
+<note version="6.3" minversion="6.2.2" severity="warning">
+Since Version 6.2.2 text objects can contain more than one line,
+which will not be processed correctly with this version.
+</note>
 <note version="8.2" severity="warning">
 Since Version 8.2, EAGLE supports online libraries. The ids

Commit message: updated
Other:
- board text added: "Designed & Manufactured by Pinwheel Robotics 01/12/2021 FutureBot Wi-Fi Shield V1.0"
- board text removed: "Designed & Manufacturd by Pinwheel Robotics 17/11/2021 FutureBot Wi-Fi Shield V1.0"
